Commit message: b2-b2w

File: source/robot_lab/data/Robots/unitree/b2_description/urdf/b2_description.urdf (robot description, URDF)
Before this commit: robot b2_description, 37 links, 36 joints
Links:
- link FL_foot: mass 0.126 -> 0.537; geometry collision box size=0.07 0.065 0.035; collision cylinder length=0.035 radius=0.1075
- link FR_foot: mass 0.126 -> 0.537; geometry collision box size=0.07 0.065 0.035; collision cylinder length=0.035 radius=0.1075
- link RL_foot: mass 0.126 -> 0.537; geometry collision box size=0.07 0.065 0.035; collision cylinder length=0.035 radius=0.1075
- link RR_foot: mass 0.126 -> 0.537; geometry collision box size=0.07 0.065 0.035; collision cylinder length=0.035 radius=0.1075

Commit message: add wheel joint

File: source/robot_lab/data/Robots/unitree/b2_description/urdf/b2_description.urdf (robot description, URDF)
Before this commit: robot b2_description, 37 links, 36 joints
Links:
- added link FL_wheel, mass 1.16; collision box size=0.07 0.065 0.035; collision mesh filename=package://unitree/b2_description/meshes/foot_wheel.STL
- added link FR_wheel, mass 1.16; collision box size=0.07 0.065 0.035; collision mesh filename=package://unitree/b2_description/meshes/foot_wheel.STL
- added link RL_wheel, mass 1.16; collision box size=0.07 0.065 0.035; collision mesh filename=package://unitree/b2_description/meshes/foot_wheel.STL
- added link RR_wheel, mass 1.16; collision box size=0.07 0.065 0.035; collision mesh filename=package://unitree/b2_description/meshes/foot_wheel.STL
- link FL_foot: mass 0.537 -> None; geometry collision sphere radius=0.032
- link FR_foot: mass 0.537 -> None; geometry collision sphere radius=0.032
- link RL_foot: mass 0.537 -> None; geometry collision sphere radius=0.032
- link RR_foot: mass 0.537 -> None; geometry collision sphere radius=0.032
Joints:
- added joint FL_wheel_to_FL_foot_joint: type fixed, parent FL_foot, child FL_wheel, origin xyz=0 0 0 rpy=0 0 0
- added joint FR_wheel_to_FR_foot_joint: type fixed, parent FR_foot, child FR_wheel, origin xyz=0 0 0 rpy=0 -1.43 3.1415
- added joint RL_wheel_to_RL_foot_joint: type fixed, parent RL_foot, child RL_wheel, origin xyz=0 0 0 rpy=0 0 0
- added joint RR_wheel_to_RR_foot_joint: type fixed, parent RR_foot, child RR_wheel, origin xyz=0 0 0 rpy=0 -1.43 3.1415

Commit message: fix collision

File: source/robot_lab/data/Robots/unitree/b2_description/urdf/b2_description.urdf (robot description, URDF)
Before this commit: robot b2_description, 41 links, 40 joints
Links:
- link FL_wheel: geometry collision mesh filename=package://unitree/b2_description/meshes/foot_connect.STL; collision mesh filename=package://unitree/b2_description/meshes/foot_wheel.STL
- link FR_wheel: geometry collision mesh filename=package://unitree/b2_description/meshes/foot_connect.STL; collision mesh filename=package://unitree/b2_description/meshes/foot_wheel.STL
- link RL_wheel: geometry collision mesh filename=package://unitree/b2_description/meshes/foot_connect.STL; collision mesh filename=package://unitree/b2_description/meshes/foot_wheel.STL
- link RR_wheel: geometry collision mesh filename=package://unitree/b2_description/meshes/foot_connect.STL; collision mesh filename=package://unitree/b2_description/meshes/foot_wheel.STL
